Commit message: 628

File: sim_mesh/franka_fr3/franka_ati_hand.urdf (robot description, URDF)
Before this commit: robot franka_ati_hand, 17 links, 16 joints
Links:
- removed link ati_hand_adapter_link
Joints:
- removed joint ft_ati_m8_joint
- joint fr3_hand_joint: origin xyz=0 0 0 rpy=0 0 -0.7853981633974483 -> xyz=0 0 0.03 rpy=0 0 -0.7853981633974483; parent ati_hand_adapter_link -> ft_ati_m8_link
